File: hw/krampus/_autosave-krampus.kicad_pcb (KiCad board)
At the start: 2 copper layers, 26.7 x 29.2 mm, 29 parts, among them J1 Conn_01x05, J2 Conn_02x03_Odd_Even, Q1 2N7002, Q2 2N7002, Q3 2N7002, Q4 Q_PMOS_GSD, U1 ESP-C3-WROOM-02, U2 TPS562200

Commit message: start board design
Routing:
- net GND: vias 9 -> 5
Changed lines of the file:
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@@
     (thickness 1.6)
     (drawings 4)
-    (tracks 130)
+    (tracks 126)
     (zones 0)
     (modules 29)
@@
   (segment (start 198.12 98.7275) (end 198.12 99.06) (width 0.25) (layer F.Cu) (net 0))
   (segment (start 196.9285 97.536) (end 198.12 98.7275) (width 0.25) (layer F.Cu) (net 0))
-  (via (at 193.929 88.011) (size 0.8) (drill 0.4) (layers F.Cu B.Cu) (net 5))
-  (via (at 193.04 88.9) (size 0.8) (drill 0.4) (layers F.Cu B.Cu) (net 5))
-  (via (at 194.818 88.9) (size 0.8) (drill 0.4) (layers F.Cu B.Cu) (net 5))
-  (via (at 193.929 89.789) (size 0.8) (drill 0.4) (layers F.Cu B.Cu) (net 5))
   (via (at 193.929 88.9) (size 0.8) (drill 0.4) (layers F.Cu B.Cu) (net 5))
   (segment (start 182.582 102.362) (end 182.582 101.856) (width 0.25) (layer F.Cu) (net 1))
