File: hw/krampus/krampus.sch (KiCad schematic (older format))
At the start: 25 parts

Commit message: updates
Parts:
- added D1: D_Zener, symbol Device:D_Zener
- added Q4: Q_PMOS_GSD, Package_TO_SOT_SMD:SOT-23, symbol Device:Q_PMOS_GSD
- added R13: 100, Resistor_SMD:R_0402_1005Metric, symbol Device:R_Small
- C1, C2: renamed from C?; value C_Small -> 22p
- J1: renamed from J?; footprint (none) -> Connector_PinHeader_1.00mm:PinHeader_1x05_P1.00mm_Vertical_SMD_Pin1Left
- R1, R10, R11, R12, R2, R3, R4, R5, R6, R7, R8, R9: renamed from R?; footprint (none) -> Resistor_SMD:R_0402_1005Metric
- gave numbers to parts that had none: 10
Connections:
- net GND: now also R13.2
- net RAW_PWR: now also Q4.3 (D); no longer C3.1, R1.1, U2.3 (VIN)
- new net: D1.2 (A), Q4.1 (G), R13.1
- new net: C3.1, D1.1 (K), Q4.2 (S), R1.1, U2.3 (VIN)

Commit message: start board design
Parts:
- removed C1, C2: 22p, symbol Device:C_Small
- removed C6: 22u, symbol Device:C_Small
- added C1: 1u, Capacitor_SMD:C_0402_1005Metric, symbol Device:C
- added D2: pwr, LED_SMD:LED_0805_2012Metric, symbol Device:LED
- added J2: Conn_02x03_Odd_Even, Connector:Tag-Connect_TC2030-IDC-NL_2x03_P1.27mm_Vertical, symbol Connector_Generic:Conn_02x03_Odd_Even
- added R14: 220, Resistor_SMD:R_0402_1005Metric, symbol Device:R_Small
- added R15: 10k, Resistor_SMD:R_0402_1005Metric, symbol Device:R
- C3: footprint (none) -> Capacitor_Tantalum_SMD:CP_EIA-3528-12_Kemet-T; mfgpart (none) -> CA45-B025K106T
- C4: footprint (none) -> Capacitor_SMD:C_0402_1005Metric; mfgpart (none) -> CL05B104KB54PNC
- C5: footprint (none) -> Capacitor_Tantalum_SMD:CP_EIA-3528-12_Kemet-T; mfgpn (none) -> TAJB226K016RNJ
- J1: footprint Connector_PinHeader_1.00mm:PinHeader_1x05_P1.00mm_Vertical_SMD_Pin1Left -> Connector_PinHeader_1.00mm:PinHeader_1x05_P1.00mm_Vertical
- L1: footprint (none) -> feet:Sunlord_MWSA0402S; mfgpart (none) -> MWSA0402S-3R3MT
Connections:
- net +3V3: now also D2.2 (A), J2.4 (Pin_4), R15.2
- net GND: now also C1.2, J2.6 (Pin_6), R14.2
- net EN: now reaches U1.2 (EN)
- net EN: now also C1.1, R15.1
- net TMS: now reaches U1.3 (IO4)
- net TMS: now also J2.5 (Pin_5)
- net TDI: now reaches U1.4 (IO5)
- net TDI: now also J2.3 (Pin_3)
- net TCK: now reaches U1.5 (IO6)
- net TCK: now also J2.1 (Pin_1)
- net TDO: now reaches U1.6 (IO7)
- net TDO: now also J2.2 (Pin_2)
- net VIN: now reaches C3.1, D1.1 (K), Q4.2 (S), R1.1, U2.3 (VIN)
- net SW: now reaches C4.1, L1.1, U2.2 (SW)
- net D+: no longer names the net of U1.14 (IO19)
- net D-: no longer names the net of U1.13 (IO18)
Other:
- note added: "power reg"
- moved on the sheet: C3, C4, C5, D1, J1, L1, Q4, R1, R13, R6, R7, U2
